File: Hardware/STM32_Motor_Kit_v0.1/STM32_Motor_Kit_v0.1.kicad_pcb (KiCad board)
At the start: 4 copper layers, 150 x 100 mm, 361 parts, among them J1 Conn_01x02_Male, J2 Conn_02x04_Odd_Even, J3 Conn_01x02_Male, J4 Conn_01x03_Male, J5 Conn_01x05_Male, J6 Conn_02x05_Odd_Even, J7 Conn_01x02_Male, J8 USB_B_Mini, Q1 NTMFS4119NT1G, Q2 NTMFS4119NT1G, Q3 NTMFS4119NT1G, Q4 NTMFS4119NT1G, Q5 NTMFS4119NT1G, Q6 NTMFS4119NT1G, Q7 MMUN2235LT1G, SW1 SW_DIP_x01, SW2 Push_Button_SMD_4P, SW3 Push_Button_SMD_4P, U1 STM32G431RBT6, U10 LMV358IDRG4, U11 LMV358IDRG4, U12 LMV358IDRG4, U13 LSF0204DPWR, U14 THVD1500D, U15 SN74HC595DRG3, U16 M24C64-WMN6TP, U17 TVS_Diode_USB, U2 AMS111733TR-HT, U3 LMV358IDRG4, U4 TPS54331DR, U5 MC78M15CDTRKG-, U6 TJA1441BT_0Z, U7 IR2104STRPBF, U8 IR2104STRPBF, U9 IR2104STRPBF, Y1 CRYSTAL_8mHz

Commit message: Added GND polygon to Inner Layer-1
Parts:
- RV1: value WH148-1A-2-20V-B1K -> WH148-1A-2-20V-B1K
- moved JP6 2.51 mm to (116.5, 84.5), turned to -90 degrees
- moved JP7 2.50 mm to (116.5, 95.0), turned to -90 degrees
- moved JP5 2.48 mm to (116.5, 105.5), turned to -90 degrees
- moved D28 0.75 mm to (169.8, 134.8)
- moved JP10 0.51 mm to (116.5, 124.5)
- moved D27 0.50 mm to (176.0, 126.5)
- moved D29 0.25 mm to (181.8, 134.8)
- moved JP8 0.12 mm to (116.5, 111.5)
- moved JP9 0.12 mm to (116.5, 117.5)
Connections:
- C43 pad 1: Net-(JP6-B) -> Net-(JP6-A)
- C44 pad 1: Net-(JP7-B) -> Net-(JP7-A)
- C45 pad 1: Net-(JP5-B) -> Net-(JP5-A)
- C46 pad 1: Net-(JP6-B) -> Net-(JP6-A)
- C47 pad 1: Net-(JP7-B) -> Net-(JP7-A)
- C48 pad 1: Net-(JP5-B) -> Net-(JP5-A)
- C49 pad 1: Net-(JP6-B) -> Net-(JP6-A)
- C50 pad 1: Net-(JP7-B) -> Net-(JP7-A)
- C51 pad 1: Net-(JP5-B) -> Net-(JP5-A)
- D12 pad 2: Net-(JP6-B) -> Net-(JP6-A)
- D13 pad 2: Net-(JP7-B) -> Net-(JP7-A)
- D14 pad 2: Net-(JP5-B) -> Net-(JP5-A)
- JP5 pad 1: +15V -> Net-(JP5-A)
- JP5 pad 2: Net-(JP5-B) -> +15V
- JP6 pad 1: +15V -> Net-(JP6-A)
- JP6 pad 2: Net-(JP6-B) -> +15V
- JP7 pad 1: +15V -> Net-(JP7-A)
- JP7 pad 2: Net-(JP7-B) -> +15V
- U7 pad 1: Net-(JP6-B) -> Net-(JP6-A)
- U8 pad 1: Net-(JP7-B) -> Net-(JP7-A)
- U9 pad 1: Net-(JP5-B) -> Net-(JP5-A)
Routing:
- net Net-(JP9-A): track 2.82 -> 15.5 mm, vias 0 -> 1
- net Net-(JP8-A): track 2.71 -> 15.4 mm, vias 0 -> 1
- net Net-(JP10-A): track 2.82 -> 15.3 mm, vias 0 -> 1
- net /Motor_Control/UVW_Phase_Total: track 105.9 -> 101.2 mm
- net /Motor_Control/W_Shunt_High: track 52.1 -> 49.2 mm
- net /Motor_Control/V_Shunt_High: track 35.0 -> 33.1 mm
- net GND: vias 29 -> 76
- net /Motor_Control/V_Phase_COM: vias 2 -> 11
- added copper zone on In1.Cu, net GND
- added copper zone on F.Cu, net Net-(JP5-A)
- added copper zone on F.Cu, net Net-(JP6-A)
- added copper zone on F.Cu, net Net-(JP7-A)
- removed copper zone on F.Cu, net Net-(JP5-B)
- removed copper zone on F.Cu, net Net-(JP6-B)
- removed copper zone on F.Cu, net Net-(JP7-B)

Commit message: Firmware Configuration added, Motor Control Pins and BackEMF Analog Pins setted.
Parts:
- moved C81 14.2 mm to (95.8, 92.8), turned to 0 degrees
- moved C82 11.9 mm to (95.8, 94.5), turned to 0 degrees
- moved C83 9.57 mm to (95.8, 96.2), turned to 0 degrees
- moved C22 3.61 mm to (95.8, 91.0)
- moved D27 2.25 mm to (176.0, 128.8)
- moved D28 1.00 mm to (169.8, 135.8)
- moved D29 1.00 mm to (181.8, 135.8)
Connections:
- C22 pad 1: /Power/BUS_Voltage_Read -> /ADC_BUS_Voltage_Read
- C81 pad 1: /Motor_Control/Shunt_ADC_U -> /ADC_Shunt_U
- C82 pad 1: /Motor_Control/Shunt_ADC_V -> /ADC_Shunt_V
- C83 pad 1: /Motor_Control/Shunt_ADC_W -> /ADC_Shunt_W
- D45 pad 1: Net-(U1A-PC0) -> Net-(D45-Pad1)
- R62 pad 1: /Motor_Control/Shunt_ADC_U -> /ADC_Shunt_U
- R63 pad 1: /Motor_Control/Shunt_ADC_V -> /ADC_Shunt_V
- R64 pad 1: /Motor_Control/Shunt_ADC_W -> /ADC_Shunt_W
- R9 pad 1: /Power/BUS_Voltage_Read -> /ADC_BUS_Voltage_Read
- TP10 pad 1: /Motor_Control/V_Drive_H -> /V_Drive_H
- TP11 pad 1: /Motor_Control/W_Drive_H -> /W_Drive_H
- TP12 pad 1: /Motor_Control/U_Drive_L -> /U_Drive_L
- TP13 pad 1: /Motor_Control/V_Drive_L -> /V_Drive_L
- TP14 pad 1: /Motor_Control/W_Drive_L -> /W_Drive_L
- TP15 pad 1: /Motor_Control/Shunt_ADC_U -> /ADC_Shunt_U
- TP16 pad 1: /Motor_Control/Shunt_ADC_V -> /ADC_Shunt_V
- TP17 pad 1: /Motor_Control/Shunt_ADC_W -> /ADC_Shunt_W
- TP3 pad 1: /Power/BUS_Voltage_Read -> /ADC_BUS_Voltage_Read
- TP33 pad 1: Net-(U1A-PC0) -> Net-(D45-Pad1)
- TP9 pad 1: /Motor_Control/U_Drive_H -> /U_Drive_H
- U1 pad 10: /MCU/PC2 -> /U_Drive_H
- U1 pad 12: /MCU/User_Button -> /MCU/PA0
- U1 pad 20: /MCU/PA6 -> /ADC_Shunt_W
- U1 pad 21: /MCU/PA7 -> /W_Drive_L
- U1 pad 22: /MCU/PC4 -> /ADC_Shunt_V
- U1 pad 23: /MCU/PC5 -> /ADC_Shunt_U
- U1 pad 24: /MCU/PB0 -> /V_Drive_L
- U1 pad 25: /MCU/PB1 -> /U_Drive_L
- U1 pad 26: /MCU/PB2 -> /ADC_BUS_Voltage_Read
- U1 pad 8: Net-(U1A-PC0) -> /W_Drive_H
- U1 pad 9: /MCU/PC1 -> /V_Drive_H
- U7 pad 2: /Motor_Control/U_Drive_H -> /U_Drive_H
- U7 pad 3: /Motor_Control/U_Drive_L -> /U_Drive_L
- U8 pad 2: /Motor_Control/V_Drive_H -> /V_Drive_H
- U8 pad 3: /Motor_Control/V_Drive_L -> /V_Drive_L
- U9 pad 2: /Motor_Control/W_Drive_H -> /W_Drive_H
- U9 pad 3: /Motor_Control/W_Drive_L -> /W_Drive_L
Routing:
- net /U_Drive_H: track 0.00 -> 60.3 mm, vias 0 -> 2
- net /W_Drive_L: track 0.00 -> 58.6 mm, vias 0 -> 2
- net /W_Drive_H: track 0.00 -> 54.2 mm, vias 0 -> 2
- net /V_Drive_H: track 0.00 -> 52.5 mm, vias 0 -> 2
- net /V_Drive_L: track 0.00 -> 50.8 mm, vias 0 -> 2
- net /U_Drive_L: track 0.00 -> 46.6 mm, vias 0 -> 2
- net /ADC_Shunt_W: track 0.00 -> 44.6 mm
- net /ADC_BUS_Voltage_Read: track 0.00 -> 41.7 mm
- net /ADC_Shunt_V: track 0.00 -> 40.3 mm
- net /ADC_Shunt_U: track 0.00 -> 36.1 mm
- net /Motor_Control/Shunt_ADC_W: track 24.7 -> 0.00 mm
- net /Motor_Control/V_Drive_H: track 23.2 -> 0.00 mm
- net /Motor_Control/W_Drive_H: track 23.1 -> 0.00 mm
- net /Motor_Control/U_Drive_H: track 22.8 -> 0.00 mm
- net /Motor_Control/W_Drive_L: track 22.7 -> 0.00 mm
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- added copper zone on B.Cu, net +3.3V

Commit message: 22.08.2024
Parts:
- added R104: 33R, AKE_Resistor_SMD:RES_0603, F.Cu at (60.0, 81.0)
- added R105: 33R, AKE_Resistor_SMD:RES_0603, F.Cu at (60.0, 79.5)
- added R106: 33R, AKE_Resistor_SMD:RES_0603, F.Cu at (60.0, 78.0)
- added R107: 33R, AKE_Resistor_SMD:RES_0603, F.Cu at (60.0, 76.5)
- added R108: 33R, AKE_Resistor_SMD:RES_0603, F.Cu at (60.0, 75.0)
- added R109: 33R, AKE_Resistor_SMD:RES_0603, F.Cu at (60.0, 73.5)
- added R110: 33R, AKE_Resistor_SMD:RES_0603, F.Cu at (60.0, 72.0)
- added R111: 33R, AKE_Resistor_SMD:RES_0603, F.Cu at (60.0, 70.5)
- added R112: 33R, AKE_Resistor_SMD:RES_0603, F.Cu at (60.0, 69.0)
- added R113: 33R, AKE_Resistor_SMD:RES_0603, F.Cu at (60.0, 67.5)
- added R114: 33R, AKE_Resistor_SMD:RES_0603, F.Cu at (60.0, 66.0)
- added R115: 33R, AKE_Resistor_SMD:RES_0603, F.Cu at (60.0, 64.5)
- added R116: 33R, AKE_Resistor_SMD:RES_0603, F.Cu at (60.0, 63.0)
- added R85: 33R, AKE_Resistor_SMD:RES_0603, F.Cu at (60.0, 84.0)
- added R86: 33R, AKE_Resistor_SMD:RES_0603, F.Cu at (60.0, 82.5)
- C4: value 100nF_50V -> 2.2uF_10V
- J6: value Conn_02x05_Odd_Even -> Conn_02x09_Odd_Even; footprint AKE_Pinheader_TH:PinHeader_2x05_P2.54mm_Vertical -> AKE_Pinheader_TH:PinHeader_2x09_P2.54mm_Vertical
- R98: value 4.7K -> 1K
- moved C5 57.5 mm to (90.8, 100.2)
- moved C6 45.8 mm to (79.2, 100.5), turned to 180 degrees
- moved TP19 44.2 mm to (121.8, 135.5), turned to 180 degrees
- moved C9 43.4 mm to (79.8, 84.8), turned to 180 degrees
- moved R71 43.1 mm to (124.5, 135.2), turned to 180 degrees
- moved R98 42.6 mm to (73.5, 76.5), turned to 90 degrees
- moved TP33 41.2 mm to (73.5, 79.0)
- moved R70 41.0 mm to (124.5, 133.8), turned to 180 degrees
- moved TP18 39.8 mm to (121.8, 133.5), turned to 180 degrees
- moved D45 39.5 mm to (71.8, 76.5)
- moved C85 26.4 mm to (71.8, 96.0), turned to 180 degrees
- moved C84 22.9 mm to (71.8, 94.5), turned to 180 degrees
- moved FID1 15.4 mm to (41.2, 54.2)
- moved J2 11.8 mm to (55.7, 95.5), turned to 180 degrees
- moved C37 11.0 mm to (76.0, 116.0)
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Connections:
- C102 pad 2: /MCU/User_Button -> /MCU/PD2
- C35 pad 1: /Programming_and_Uart/FTDI_UART_TX -> /MCU/PA9
- C36 pad 1: /Programming_and_Uart/FTDI_UART_RX -> /MCU/PA10
- C37 pad 1: /CanBus_Communication/MCU_CAN_TX -> /MCU_CAN_TX
- C84 pad 1: /Encoder/ENC_CLK_A -> /ENC_CLK_A
- C85 pad 1: /Encoder/ENC_DATA_B -> /ENC_DATA_B
- C98 pad 1: /Potentiometer/Potentiometer_Read -> /Potentiometer_Read
- D37 pad 1: /Potentiometer/Potentiometer_Read -> /Potentiometer_Read
- D45 pad 1: Net-(D45-Pad1) -> GND
- D9 pad 2: Net-(J2-Pin_2) -> Net-(J2-Pin_8)
- J2 pad 1: GND -> /MCU/SWCLK
- J2 pad 2: Net-(J2-Pin_2) -> /MCU/RST
- J2 pad 3: GND -> /MCU/SWDIO
- J2 pad 4: /MCU/RST -> GND
- J2 pad 6: /MCU/SWDIO -> GND
- J2 pad 8: /MCU/SWCLK -> Net-(J2-Pin_8)
- J6 pad 1: unconnected-(J6-Pin_1-Pad1) -> /GPIO/Pin_1
- J6 pad 10: unconnected-(J6-Pin_10-Pad10) -> /GPIO/Pin_10
- J6 pad 2: unconnected-(J6-Pin_2-Pad2) -> /GPIO/Pin_2
- J6 pad 3: unconnected-(J6-Pin_3-Pad3) -> /GPIO/Pin_3
- J6 pad 4: unconnected-(J6-Pin_4-Pad4) -> /GPIO/Pin_4
- J6 pad 5: unconnected-(J6-Pin_5-Pad5) -> /GPIO/Pin_5
- J6 pad 6: unconnected-(J6-Pin_6-Pad6) -> /GPIO/Pin_6
- J6 pad 7: unconnected-(J6-Pin_7-Pad7) -> /GPIO/Pin_7
- J6 pad 8: unconnected-(J6-Pin_8-Pad8) -> /GPIO/Pin_8
- J6 pad 9: unconnected-(J6-Pin_9-Pad9) -> /GPIO/Pin_9
- R1 pad 2: /MCU/BOOT -> /MCU_CAN_RX
- R103 pad 1: /MCU/User_Button -> /MCU/PD2
- R19 pad 2: /Programming_and_Uart/FTDI_UART_TX -> /MCU/PA9
- R20 pad 2: /Programming_and_Uart/FTDI_UART_RX -> /MCU/PA10
- R21 pad 1: /CanBus_Communication/MCU_CAN_RX -> /MCU_CAN_RX
- R70 pad 2: /Encoder/ENC_DATA_B -> /ENC_DATA_B
- R71 pad 2: /Encoder/ENC_CLK_A -> /ENC_CLK_A
- R80 pad 2: /RS485_Communication/RS485_RX -> /USART2_TX
- R81 pad 2: /RS485_Communication/RS485_ENABLE -> /MCU/PB10
- R82 pad 2: /RS485_Communication/RS485_TX -> /USART2_RX
- R89 pad 2: /Potentiometer/Potentiometer_Read -> /Potentiometer_Read
- R98 pad 1: Net-(D45-Pad2) -> /MCU/PA8
- R98 pad 2: +3.3V_MCU -> Net-(D45-Pad2)
- SW1 pad 1: /MCU/BOOT -> /MCU_CAN_RX
- SW3 pad 1: /MCU/User_Button -> /MCU/PD2
- SW3 pad 2: /MCU/User_Button -> /MCU/PD2
- TP18 pad 1: /Encoder/ENC_DATA_B -> /ENC_DATA_B
- TP19 pad 1: /Encoder/ENC_CLK_A -> /ENC_CLK_A
- TP20 pad 1: /RS485_Communication/RS485_RX -> /USART2_TX
- TP21 pad 1: /RS485_Communication/RS485_ENABLE -> /MCU/PB10
- TP22 pad 1: /RS485_Communication/RS485_TX -> /USART2_RX
- TP23 pad 1: /Potentiometer/Potentiometer_Read -> /Potentiometer_Read
- TP33 pad 1: Net-(D45-Pad1) -> /MCU/PA8
- TP7 pad 1: /CanBus_Communication/MCU_CAN_TX -> /MCU_CAN_TX
- TP8 pad 1: /CanBus_Communication/MCU_CAN_RX -> /MCU_CAN_RX
- U1 pad 11: /MCU/PC3 -> /Potentiometer_Read
- U1 pad 14: /MCU/PA2 -> /USART2_TX
- U1 pad 17: /MCU/PA3 -> /USART2_RX
- U1 pad 2: /MCU/PC13 -> /LED_OUT/SN74HC_OE
- U1 pad 39: /MCU/PC7 -> /Flash_IC/FLASH_WC
- U1 pad 40: /MCU/PC8 -> /Flash_IC/FLASH_I2C_CLK
- U1 pad 41: /MCU/PC9 -> /Flash_IC/FLASH_I2C_SDA
- U1 pad 51: /MCU/PA15 -> /LED_OUT/SPI_CS
- U1 pad 56: /MCU/PB3 -> /LED_OUT/SPI_CLK
- U1 pad 57: /MCU/PB4 -> /LED_OUT/SPI_MISO
- U1 pad 58: /MCU/PB5 -> /LED_OUT/SPI_MOSI
- U1 pad 59: /MCU/PB6 -> /ENC_CLK_A
- U1 pad 60: /MCU/PB7 -> /ENC_DATA_B
- U1 pad 61: /MCU/BOOT -> /MCU_CAN_RX
- U1 pad 62: /MCU/PB9 -> /MCU_CAN_TX
- U6 pad 1: /CanBus_Communication/MCU_CAN_TX -> /MCU_CAN_TX
Routing:
- net /LED_OUT/SPI_CS: track 5.45 -> 63.9 mm
- net /ENC_CLK_A: track 0.00 -> 57.5 mm, vias 0 -> 1
- net /LED_OUT/SPI_MISO: track 5.37 -> 62.6 mm
- net /Potentiometer_Read: track 0.00 -> 55.9 mm, vias 0 -> 2
- net /LED_OUT/SPI_CLK: track 5.00 -> 60.9 mm
- net /ENC_DATA_B: track 0.00 -> 55.9 mm, vias 0 -> 1
- net /LED_OUT/SPI_MOSI: track 5.37 -> 57.8 mm, vias 0 -> 2
- net /MCU/PD2: track 0.00 -> 52.0 mm, vias 0 -> 2
- net Net-(U13-A3): track 50.7 -> 2.70 mm
- net Net-(U13-A2): track 50.2 -> 2.35 mm
- net /LED_OUT/SN74HC_OE: track 12.0 -> 59.7 mm, vias 0 -> 2
- net /MCU_CAN_RX: track 0.00 -> 42.3 mm, vias 0 -> 3
- net /Potentiometer/Potentiometer_Read: track 38.4 -> 0.00 mm
- net /MCU_CAN_TX: track 0.00 -> 35.9 mm
- net /MCU/PA9: track 0.00 -> 29.2 mm
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- added copper zone on B.Cu, net +5V
- added copper zone on F.Cu, net Net-(J2-Pin_8)

Commit message: 23.08.2024
Parts:
- R6: value 1K -> 10K
- moved C10 59.2 mm to (95.8, 87.0), turned to 180 degrees
- moved C7 59.1 mm to (95.8, 88.5), turned to 180 degrees
- moved C8 59.1 mm to (95.8, 90.0), turned to 180 degrees
- moved R85 21.0 mm to (60.0, 63.0)
- moved R86 18.0 mm to (60.0, 64.5)
- moved R104 15.0 mm to (60.0, 66.0)
- moved R115 15.0 mm to (60.0, 79.5)
- moved R116 15.0 mm to (60.0, 78.0)
- moved R105 10.5 mm to (60.0, 69.0)
- moved R108 9.00 mm to (60.0, 84.0)
- moved STM32_Motor_Kit_v1.1 6.27 mm to (21.5, 114.5)
- moved JP1 6.08 mm to (97.0, 84.0), turned to -90 degrees
- moved R111 6.00 mm to (60.0, 76.5)
- moved R112 6.00 mm to (60.0, 75.0)
- moved C2 5.26 mm to (82.0, 103.8)
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Connections:
- R104 pad 2: /GPIO/Pin_3 -> /GPIO/Pin_13
- R105 pad 2: /GPIO/Pin_4 -> /GPIO/Pin_11
- R106 pad 2: /GPIO/Pin_5 -> /GPIO/Pin_2
- R107 pad 2: /GPIO/Pin_6 -> /GPIO/Pin_3
- R108 pad 2: /GPIO/Pin_7 -> /GPIO/Pin_1
- R109 pad 2: /GPIO/Pin_8 -> /GPIO/Pin_9
- R110 pad 2: /GPIO/Pin_9 -> /GPIO/Pin_8
- R111 pad 2: /GPIO/Pin_10 -> /GPIO/Pin_6
- R112 pad 2: /GPIO/Pin_11 -> /GPIO/Pin_7
- R114 pad 2: /GPIO/Pin_13 -> /GPIO/Pin_10
- R115 pad 2: /GPIO/Pin_14 -> /GPIO/Pin_4
- R116 pad 2: /GPIO/Pin_15 -> /GPIO/Pin_5
- R85 pad 2: /GPIO/Pin_1 -> /GPIO/Pin_15
- R86 pad 2: /GPIO/Pin_2 -> /GPIO/Pin_14
Routing:
- net +24V: track 5.07 -> 51.9 mm, vias 0 -> 1
- net /MCU/PA5: track 0.00 -> 44.4 mm, vias 0 -> 2
- net /MCU/PA4: track 0.00 -> 43.2 mm, vias 0 -> 2
- net /MCU/PA1: track 0.00 -> 40.3 mm, vias 0 -> 2
- net /MCU/PA0: track 0.00 -> 38.5 mm, vias 0 -> 2
- net /MCU/PC6: track 0.00 -> 37.1 mm, vias 0 -> 2
- net /ENC_CLK_A: track 57.5 -> 90.8 mm, vias 1 -> 2
- net /ENC_DATA_B: track 55.9 -> 87.5 mm, vias 1 -> 2
- net /MCU/PB10: track 2.61 -> 32.9 mm, vias 0 -> 2
- net /MCU/PC15: track 10.9 -> 34.9 mm, vias 0 -> 2
- net /MCU/PC14: track 9.34 -> 32.6 mm, vias 0 -> 2
- net /MCU/PC10: track 0.00 -> 22.8 mm, vias 0 -> 2
- net /MCU/PC11: track 0.00 -> 22.3 mm, vias 0 -> 2
- net /MCU/PC12: track 0.00 -> 22.2 mm, vias 0 -> 2
- net GND: track 69.5 -> 91.5 mm, vias 148 -> 155
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