File: Hardware/STM32_Motor_Kit_v0.1/STM32_Motor_Kit_v0.1.kicad_pcb (KiCad board)
At the start: 4 copper layers, 150 x 100 mm, 403 parts, among them J1 Conn_01x02_Male, J2 Conn_02x04_Odd_Even, J3 Conn_01x02_Male, J4 Conn_01x03_Male, J5 Conn_01x06_Male, J6 Conn_02x09_Odd_Even, J7 Conn_01x02_Male, J8 USB_B_Mini, Q1 NTMFS4119NT1G, Q2 NTMFS4119NT1G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

Commit message: 23.02.2026
Parts:
- moved FID2 15.3 mm to (191.2, 60.0)
Routing:
- net GND: vias 597 -> 599
