File: Hardware/STM32_Motor_Kit_v0.1/GPIO.kicad_sch (KiCad schematic)
At the start: 1 part, among them J6 Conn_02x05_Odd_Even

Commit message: 22.08.2024
Parts:
- removed J6: Conn_02x05_Odd_Even, AKE_Pinheader_TH:PinHeader_2x05_P2.54mm_Vertical, symbol AKE_Connector_Pinheader:Conn_02x05_Odd_Even
- added J6: Conn_02x09_Odd_Even, AKE_Pinheader_TH:PinHeader_2x09_P2.54mm_Vertical, symbol AKE_Connector_Pinheader:Conn_02x09_Odd_Even
Connections:
- new net +3.3V: J6.18 (Pin_18)
- new net +5V: J6.17 (Pin_17)
- new net GND: J6.16 (Pin_16)
- new net Pin_1: J6.1 (Pin_1)
- new net Pin_10: J6.10 (Pin_10)
- new net Pin_11: J6.11 (Pin_11)
- new net Pin_12: J6.12 (Pin_12)
- new net Pin_13: J6.13 (Pin_13)
- new net Pin_14: J6.14 (Pin_14)
- new net Pin_15: J6.15 (Pin_15)
- new net Pin_2: J6.2 (Pin_2)
- new net Pin_3: J6.3 (Pin_3)
- new net Pin_4: J6.4 (Pin_4)
- new net Pin_5: J6.5 (Pin_5)
- new net Pin_6: J6.6 (Pin_6)
- new net Pin_7: J6.7 (Pin_7)
- new net Pin_8: J6.8 (Pin_8)
- new net Pin_9: J6.9 (Pin_9)

Commit message: 16.09.2024
Connections:
- net Pin_7 is gone; now on net GND: J6.7 (Pin_7)
Changed lines of the file:
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@@
+	(wire
+		(pts
+			(xy 87.63 101.6) (xy 83.82 101.6)
+		)
+		(stroke
+			(width 0)
+			(type default)
+		)
+	)
 	(wire
 		(pts
@@
 	(wire
 		(pts
-			(xy 83.82 101.6) (xy 87.63 101.6)
-		)
-		(stroke
-			(width 0)
-			(type default)
-		)
-	)
-	(wire
-		(pts
 			(xy 83.82 93.98) (xy 87.63 93.98)
 		)
@@
 			)
 			(justify left)
-		)
-	)
-	(hierarchical_label "Pin_7"
-		(shape input)
-		(at 83.82 101.6 180)
-		(fields_autoplaced yes)
-		(effects
-			(font
-				(size 1.27 1.27)
-			)
-			(justify right)
 		)
 	)
@@
 					(unit 1)
 				)
+			)
+		)
+	)
+	(symbol
+		(lib_id "AKE_Power:GND")
+		(at 83.82 101.6 270)
+		(unit 1)
+		(exclude_from_sim no)
+		(in_bom yes)
+		(on_board yes)
+		(dnp no)
+		(property "Reference" "#PWR0113"
+			(at 77.47 101.6 0)
+			(effects
+				(font
+					(size 1.27 1.27)
+				)
+				(hide yes)
+			)
+		)
+		(property "Value" "GND"
+			(at 78.74 101.6 90)
+			(effects
+				(font
+					(size 1.27 1.27)
+				)
+			)
+		)
+		(property "Footprint" ""
+			(at 83.82 101.6 0)
+			(effects
+				(font
+					(size 1.27 1.27)
+				)
+				(hide yes)
+			)
+		)
+		(property "Datasheet" ""
+			(at 83.82 101.6 0)
+			(effects
+				(font
+					(size 1.27 1.27)
+				)
+				(hide yes)
+			)
+		)
+		(property "Description" ""
+			(at 83.82 101.6 0)
+			(effects
+				(font
+					(size 1.27 1.27)
+				)
+				(hide yes)
+			)
+		)
+		(pin "1"
+		)
+		(instances
+			(project "STM32_Motor_Kit_v0.1"
+				(path "/350b6aea-94d6-460b-86d9-ade6c51fbb19/b50d19b9-c0b5-4836-8d49-6fa6eb4e0e8f"
+					(reference "#PWR0113")
+					(unit 1)
+				)

Commit message: 12.01.2025
Changed lines of the file:
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@@
 			(effects
 				(font
-					(size 1.27 1.27)
+					(face "Arial")
+					(size 0.635 0.635)
 				)
 				(hide yes)
@@
 			(effects
 				(font
-					(size 1.27 1.27)
+					(face "Arial")
+					(size 0.635 0.635)
 				)
 				(hide yes)
@@
 			(effects
 				(font
-					(size 1.27 1.27)
+					(face "Arial")
+					(size 0.635 0.635)
 				)
 				(hide yes)
@@
 			(effects
 				(font
-					(size 1.27 1.27)
+					(face "Arial")
+					(size 0.635 0.635)
 				)
 			)
@@
 			(effects
 				(font
-					(size 1.27 1.27)
-				)
-				(hide yes)
+					(face "Arial")
+					(size 0.635 0.635)
+				)
+				(hide yes)
