File: Hardware/STM32_Motor_Kit_v0.1/Potentiometer.kicad_sch (KiCad schematic)
At the start: 8 parts

Commit message: Added GND polygon to Inner Layer-1
Parts:
- RV1: value WH148-1A-2-20V-B1K -> WH148-1A-2-20V-B1K
Changed lines of the file:
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@@
 			)
 		)
-		(property "Value" "WH148-1A-2-20V-B1K "
+		(property "Value" "WH148-1A-2-20V-B1K"
 			(at 113.03 88.8999 0)
 			(effects

Commit message: 29.08.2024
Connections:
- net Potentiometer_Read: no longer D37.1
- net at R89.1, RV1.2: now also D37.1
Other:
- moved on the sheet: C98, D37, R89, TP23, TP24

Commit message: 12.01.2025
Changed lines of the file:
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@@
 			(effects
 				(font
-					(size 1.27 1.27)
+					(face "Arial")
+					(size 0.635 0.635)
 				)
 				(hide yes)
@@
 			(effects
 				(font
-					(size 1.27 1.27)
+					(face "Arial")
+					(size 0.635 0.635)
 				)
 				(justify left)
@@
 			(effects
 				(font
-					(size 1.27 1.27)
+					(face "Arial")
+					(size 0.635 0.635)
 				)
 				(hide yes)
@@
 			(effects
 				(font
-					(size 1.27 1.27)
+					(face "Arial")
+					(size 0.635 0.635)
 				)
 				(justify right)
@@
 			(effects
 				(font
-					(size 1.27 1.27)
+					(face "Arial")
+					(size 0.635 0.635)
 				)
 			)
@@
 			(effects
 				(font
-					(size 1.27 1.27)
+					(face "Arial")
+					(size 0.635 0.635)
 				)
 				(justify left)
@@
 			(effects
 				(font
-					(size 1.27 1.27)
+					(face "Arial")
+					(size 0.635 0.635)
 				)
 				(hide yes)
@@
 			(effects
 				(font
-					(size 1.27 1.27)
+					(face "Arial")
+					(size 0.635 0.635)
 				)
 			)
@@
 			(effects
 				(font
-					(size 1.27 1.27)
+					(face "Arial")
+					(size 0.635 0.635)
 				)
 				(hide yes)
@@
 			(effects
 				(font
-					(size 1.27 1.27)
+					(face "Arial")
+					(size 0.635 0.635)
 				)
 				(justify left)
@@
 			(effects
 				(font
-					(size 1.27 1.27)
+					(face "Arial")
+					(size 0.635 0.635)
 				)
 				(justify left)
@@
 			(effects
 				(font
-					(size 1.27 1.27)
+					(face "Arial")
+					(size 0.635 0.635)
 				)
 				(hide yes)
@@
 			(effects
 				(font
-					(size 1.27 1.27)
+					(face "Arial")
+					(size 0.635 0.635)
 				)
 				(justify left)
