File: Hardware/STM32_Motor_Kit_v0.1/RS485_Communication.kicad_sch (KiCad schematic)
At the start: 22 parts, among them J7 Conn_01x02_Male, U14 THVD1500D

Commit message: 29.08.2024
Connections:
- net +5V: no longer R84.2
- net at C92.1, JP13.1 (A), U14.8 (VCC): now also R84.2
Other:
- moved on the sheet: C92, JP13, R84

Commit message: 01.09.2024
Parts:
- added R117: 10K, AKE_Resistor_SMD:RES_0603, symbol AKE_Resistor:Resistor_US
Connections:
- net GND: now also R117.1
- net at R81.1, U14.2 (~{RE}), U14.3 (DE): now also R117.2
Other:
- moved on the sheet: R84
Changed lines of the file:
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@@
+	)
+	(junction
+		(at 129.54 73.66)
+		(diameter 0)
+		(color 0 0 0 0)
 	)
 	(junction
@@
 	)
 	(junction
+		(at 129.54 82.55)
+		(diameter 0)
+		(color 0 0 0 0)
+	)
+	(junction
 		(at 88.9 77.47)
 		(diameter 0)
@@
 	)
 	(junction
-		(at 135.89 77.47)
+		(at 129.54 77.47)
 		(diameter 0)
 		(color 0 0 0 0)
@@
 	)
 	(junction
-		(at 135.89 73.66)
-		(diameter 0)
-		(color 0 0 0 0)
-	)
-	(junction
 		(at 82.55 73.66)
 		(diameter 0)
@@
 	(wire
 		(pts
-			(xy 111.76 77.47) (xy 135.89 77.47)
+			(xy 111.76 77.47) (xy 129.54 77.47)
 		)
 		(stroke
@@
 	(wire
 		(pts
-			(xy 135.89 73.66) (xy 138.43 73.66)
-		)
-		(stroke
-			(width 0)
-			(type default)
-		)
-	)
-	(wire
-		(pts
 			(xy 240.03 81.28) (xy 260.35 81.28)
 		)
@@
 	(wire
 		(pts
-			(xy 138.43 77.47) (xy 135.89 77.47)
-		)
-		(stroke
-			(width 0)
-			(type default)
-		)
-	)
-	(wire
-		(pts
 			(xy 190.5 86.36) (xy 203.2 86.36)
 		)
@@
 	(wire
 		(pts
-			(xy 138.43 82.55) (xy 135.89 82.55)
+			(xy 138.43 82.55) (xy 129.54 82.55)
 		)
 		(stroke
@@
 	(wire
 		(pts
+			(xy 129.54 96.52) (xy 129.54 100.33)
+		)
+		(stroke
+			(width 0)
+			(type default)
+		)
+	)
+	(wire
+		(pts
 			(xy 80.01 86.36) (xy 95.25 86.36)
 		)
@@
 	(wire
 		(pts
+			(xy 129.54 73.66) (xy 138.43 73.66)
+		)
+		(stroke
+			(width 0)
+			(type default)
+		)
+	)
+	(wire
+		(pts
 			(xy 173.99 81.28) (xy 173.99 86.36)
 		)
@@
 	(wire
 		(pts
-			(xy 135.89 57.15) (xy 135.89 60.96)
+			(xy 129.54 57.15) (xy 129.54 62.23)
 		)
 		(stroke
@@
 	(wire
 		(pts
-			(xy 111.76 73.66) (xy 135.89 73.66)
+			(xy 111.76 73.66) (xy 129.54 73.66)
 		)
 		(stroke
@@
 	(wire
 		(pts
+			(xy 129.54 77.47) (xy 138.43 77.47)
+		)
+		(stroke
+			(width 0)
+			(type default)
+		)
+	)
+	(wire
+		(pts
 			(xy 240.03 74.93) (xy 236.22 74.93)
 		)
@@
 	(wire
 		(pts
-			(xy 135.89 57.15) (xy 162.56 57.15)
+			(xy 129.54 57.15) (xy 162.56 57.15)
 		)
 		(stroke
@@
 	(wire
 		(pts
+			(xy 129.54 82.55) (xy 129.54 91.44)
+		)
+		(stroke
+			(width 0)
+			(type default)
+		)
+	)
+	(wire
+		(pts
 			(xy 203.2 86.36) (xy 203.2 91.44)
 		)
@@
 	(wire
 		(pts
-			(xy 135.89 66.04) (xy 135.89 73.66)
+			(xy 129.54 67.31) (xy 129.54 73.66)
 		)
 		(stroke
@@
 	(wire
 		(pts
-			(xy 135.89 82.55) (xy 135.89 77.47)
+			(xy 129.54 82.55) (xy 129.54 77.47)
 		)
 		(stroke
@@
 	)
 	(symbol
+		(lib_id "AKE_Resistor:Resistor_US")
+		(at 129.54 93.98 180)
+		(unit 1)
+		(exclude_from_sim no)
+		(in_bom yes)
+		(on_board yes)
+		(dnp no)
+		(property "Reference" "R117"
+			(at 132.588 96.266 0)
+			(effects
+				(font
+					(size 1.27 1.27)
+				)
+			)
+		)
+		(property "Value" "10K"
+			(at 127.508 94.488 90)
+			(effects
+				(font
+					(size 1.27 1.27)
+				)
+			)
+		)
+		(property "Footprint" "AKE_Resistor_SMD:RES_0603"
+			(at 129.54 93.98 0)
+			(effects
+				(font
+					(size 1.27 1.27)
+				)
+				(hide yes)
+			)
+		)
+		(property "Datasheet" "~"
+			(at 129.54 93.98 0)
+			(effects
+				(font
+					(size 1.27 1.27)
+				)
+				(hide yes)
+			)
+		)
+		(property "Description" ""
+			(at 129.54 93.98 0)
+			(effects
+				(font
+					(size 1.27 1.27)
+				)
+				(hide yes)
+			)
+		)
+		(property "MFG P/N" "*"
+			(at 125.73 96.52 0)
+			(effects
+				(font
+					(size 1.27 1.27)
+				)
+				(hide yes)
+			)
+		)
+		(pin "1"
+		)
+		(pin "2"
+		)
+		(instances
+			(project "STM32_Motor_Kit_v0.1"
+				(path "/350b6aea-94d6-460b-86d9-ade6c51fbb19/cedb2968-52cc-413b-b98f-5f1bfed36cb3"
+					(reference "R117")
+					(unit 1)
+				)
+			)
+		)
+	)
+	(symbol
 		(lib_id "AKE_Diode:Diode_TVS_Bidirectional")
 		(at 223.52 85.09 90)
@@
 	)
 	(symbol
+		(lib_id "AKE_Power:GND")
+		(at 129.54 100.33 0)
+		(unit 1)
+		(exclude_from_sim no)
+		(in_bom yes)
+		(on_board yes)
+		(dnp no)
+		(property "Reference" "#PWR052"
+			(at 129.54 106.68 0)
+			(effects
+				(font
+					(size 1.27 1.27)
+				)
+				(hide yes)
+			)
+		)
+		(property "Value" "GND"
+			(at 129.667 104.7242 0)
+			(effects
+				(font
+					(size 1.27 1.27)
+				)
+			)
+		)
+		(property "Footprint" ""
+			(at 129.54 100.33 0)
+			(effects
+				(font
+					(size 1.27 1.27)
+				)
+				(hide yes)
+			)
+		)
+		(property "Datasheet" ""
+			(at 129.54 100.33 0)
+			(effects
+				(font
+					(size 1.27 1.27)
+				)
+				(hide yes)
+			)
+		)
+		(property "Description" ""
+			(at 129.54 100.33 0)
+			(effects
+				(font
+					(size 1.27 1.27)
+				)
+				(hide yes)
+			)
+		)
+		(pin "1"
+		)
+		(instances
+			(project "STM32_Motor_Kit_v0.1"
+				(path "/350b6aea-94d6-460b-86d9-ade6c51fbb19/cedb2968-52cc-413b-b98f-5f1bfed36cb3"
+					(reference "#PWR052")
+					(unit 1)
+				)
+			)
+		)
+	)
+	(symbol
 		(lib_id "AKE_Device:Test_Point")
 		(at 88.9 72.39 0)
@@
 	(symbol
 		(lib_id "AKE_Resistor:Resistor_US")
-		(at 135.89 63.5 180)
+		(at 129.54 64.77 180)
 		(unit 1)
 		(exclude_from_sim no)
@@
 		(dnp no)
 		(property "Reference" "R84"
-			(at 138.938 65.786 0)
+			(at 132.588 67.056 0)
 			(effects
 				(font
@@
 		)
 		(property "Value" "10K"
-			(at 133.858 64.008 90)
+			(at 127.508 65.278 90)
 			(effects
 				(font
@@
 		)
 		(property "Footprint" "AKE_Resistor_SMD:RES_0603"
-			(at 135.89 63.5 0)
+			(at 129.54 64.77 0)
 			(effects
 				(font
@@
 		)
 		(property "Datasheet" "~"
-			(at 135.89 63.5 0)
+			(at 129.54 64.77 0)
 			(effects
 				(font
@@
 		)
 		(property "Description" ""
-			(at 135.89 63.5 0)
+			(at 129.54 64.77 0)
 			(effects
 				(font
@@
 		)
 		(property "MFG P/N" "*"
-			(at 132.08 66.04 0)
-			(effects
-				(font
+			(at 125.73 67.31 0)
+			(effects
+				(font

Commit message: 12.01.2025
Changed lines of the file:
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@@
 			(effects
 				(font
-					(size 1.27 1.27)
+					(face "Arial")
+					(size 0.635 0.635)
 				)
 			)
@@
 			(effects
 				(font
-					(size 1.27 1.27)
+					(face "Arial")
+					(size 0.635 0.635)
 				)
 				(justify left)
@@
 			(effects
 				(font
-					(size 1.27 1.27)
+					(face "Arial")
+					(size 0.635 0.635)
 				)
 			)
@@
 			(effects
 				(font
-					(size 1.27 1.27)
+					(face "Arial")
+					(size 0.635 0.635)
 				)
 				(justify right)
@@
 			(effects
 				(font
-					(size 1.27 1.27)
+					(face "Arial")
+					(size 0.635 0.635)
 				)
 				(justify left)
@@
 			(effects
 				(font
-					(size 1.27 1.27)
+					(face "Arial")
+					(size 0.635 0.635)
 				)
 			)
@@
 			(effects
 				(font
-					(size 1.27 1.27)
+					(face "Arial")
+					(size 0.635 0.635)
 				)
 				(justify left)
@@
 			(effects
 				(font
-					(size 1.27 1.27)
+					(face "Arial")
+					(size 0.635 0.635)
 				)
 			)
@@
 			(effects
 				(font
-					(size 1.27 1.27)
+					(face "Arial")
+					(size 0.635 0.635)
 				)
 			)
@@
 			(effects
 				(font
-					(size 1.27 1.27)
+					(face "Arial")
+					(size 0.635 0.635)
 				)
 				(justify left)
@@
 			(effects
 				(font
-					(size 1.27 1.27)
+					(face "Arial")
+					(size 0.635 0.635)
 				)
 				(hide yes)
@@
 			(effects
 				(font
-					(size 1.27 1.27)
+					(face "Arial")
+					(size 0.635 0.635)
 				)
 				(hide yes)
@@
 			(effects
 				(font
-					(size 1.27 1.27)
+					(face "Arial")
+					(size 0.635 0.635)
 				)
 				(justify left)
@@
 			(effects
 				(font
-					(size 1.27 1.27)
+					(face "Arial")
+					(size 0.635 0.635)
 				)
 			)
@@
 			(effects
 				(font
-					(size 1.27 1.27)
+					(face "Arial")
+					(size 0.635 0.635)
 				)
 				(justify right)
@@
 			(effects
 				(font
-					(size 1.27 1.27)
+					(face "Arial")
+					(size 0.635 0.635)
 				)
 				(hide yes)
@@
 			(effects
 				(font
-					(size 1.27 1.27)
+					(face "Arial")
+					(size 0.635 0.635)
 				)
 				(hide yes)
@@
 			(effects
 				(font
-					(size 1.27 1.27)
+					(face "Arial")
+					(size 0.635 0.635)
 				)
 			)
@@
 			(effects
 				(font
-					(size 1.27 1.27)
+					(face "Arial")
+					(size 0.635 0.635)
 				)
 				(hide yes)
@@
 			(effects
 				(font
-					(size 1.27 1.27)
+					(face "Arial")
+					(size 0.635 0.635)
 				)
 				(hide yes)
@@
 			(effects
 				(font
-					(size 1.27 1.27)
+					(face "Arial")
+					(size 0.635 0.635)
 				)
 			)
@@
 			(effects
 				(font
-					(size 1.27 1.27)
+					(face "Arial")
+					(size 0.635 0.635)
 				)
 				(justify left)
@@
 			(effects
 				(font
-					(size 1.27 1.27)
+					(face "Arial")
+					(size 0.635 0.635)
 				)
 				(justify right)
@@
 			(effects
 				(font
-					(size 1.27 1.27)
+					(face "Arial")
+					(size 0.635 0.635)
 				)
 				(justify left)
@@
 			(effects
 				(font
-					(size 1.27 1.27)
+					(face "Arial")
+					(size 0.635 0.635)
 				)
 				(justify left)
@@
 			(effects
 				(font
-					(size 1.27 1.27)
+					(face "Arial")
+					(size 0.635 0.635)
 				)
 				(hide yes)
@@
 			(effects
 				(font
-					(size 1.27 1.27)
+					(face "Arial")
+					(size 0.635 0.635)
 				)
 			)
@@
 			(effects
 				(font
-					(size 1.27 1.27)
+					(face "Arial")
+					(size 0.635 0.635)
 				)
 				(hide yes)
@@
 			(effects
 				(font
-					(size 1.27 1.27)
+					(face "Arial")
+					(size 0.635 0.635)
 				)
 			)
@@
 			(effects
 				(font
-					(size 1.27 1.27)
+					(face "Arial")
+					(size 0.635 0.635)
 				)
 			)
@@
 			(effects
 				(font
-					(size 1.27 1.27)
+					(face "Arial")
+					(size 0.635 0.635)
 				)
 				(justify left)

Commit message: Şema üzerinde değişiklikler devam ediyor
Parts:
- removed C96: 1nF_50V, AKE_Capacitor_SMD:CAP_0603, symbol AKE_Capacitor:Capacitor_UnPolarised
- removed FB1, FB2: LCB1608-121Y-N, AKE_Resistor_SMD:RES_0603, symbol AKE_Inductor:Ferrite_Bead
- removed TH2, TH3: KMC1S010RY, AKE_Resistor_SMD:RES_0603, symbol AKE_NTC_PTC:PTC_Thermistor_US
- added D34: PESD2CANFD27V-TR, AKE_Diode_SMD:SOT-23, symbol DC_DCU_v0.1-rescue:PESD2CANFD27V-TR-AKE_Diode
- added JP11: Jumper_Pinheader, AKE_Pinheader_TH:PinHeader_1x02_P2.54mm_Vertical, symbol AKE_Device:Jumper_Pinheader
- added L8: PE-1206CCMC222STS, MN_Inductor_SMD:CMC_1206_4_LEAD, symbol MN_Inductor:PE-1206CCMC222STS
- added R131, R132: 1K, AKE_Resistor_SMD:RES_0603, symbol AKE_Resistor:Resistor_US
Connections:
- net RS485_1_N is gone; now on net RS485_0_N: C95.2, D36.2, R87.2
- net +5V: now also R131.2
- net GND: now also D34.3, R132.1
- net RS485_0_N: now also D34.2, L8.2, R131.1
- net RS485_0_P: now also C97.2, D36.1, D34.1, JP11.1 (A), L8.3, R132.2
- net RS485_2_N: now also L8.1
- net RS485_2_P: now also L8.4
- removed net RS485_1_P: C97.2, D36.1, R87.1
- new net: JP11.2 (B), R87.1
Other:
- moved on the sheet: C92, C93, C94, C95, C97, D36, J7, JP13, R117, R80, R81, R82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
