File: Hardware/STM32_Motor_Kit_v0.1/User_Command.kicad_sch (KiCad schematic)
At the start: 6 parts, among them J2 Conn_02x04_Odd_Even

Commit message: 22.08.2024
Parts:
- removed C35, C36: 100pF_50V, AKE_Capacitor_SMD:CAP_0603, symbol AKE_Capacitor:Capacitor_UnPolarised
- removed D9: B0520LW-7-F, AKE_Diode_SMD:SOD-123, symbol AKE_Diode:Diode_Schottky
- removed J2: Conn_02x04_Odd_Even, AKE_Pinheader_TH:PinHeader_2x04_P2.54mm_Vertical, symbol AKE_Connector_Pinheader:Conn_02x04_Odd_Even
- removed R19, R20: 47R, AKE_Resistor_SMD:RES_0603, symbol AKE_Resistor:Resistor_US
- added C102: 100nF_50V, AKE_Capacitor_SMD:CAP_0603, symbol AKE_Capacitor:Capacitor_UnPolarised
- added D45: Blue, AKE_Led_SMD:LED_0805, symbol AKE_Diode:Diode_LED
- added R103: 10K, AKE_Resistor_SMD:RES_0603, symbol AKE_Resistor:Resistor_US
- added R98: 1K, AKE_Resistor_SMD:RES_0603, symbol AKE_Resistor:Resistor_US
- added SW3: Push_Button_SMD_4P, AKE_Button_SMD_TH:SW_PTS645SK50SMTR92, symbol AKE_Device:Push_Button_SMD_4P
- added TP33: Test_Point, AKE_PCB:TEST_POINT, symbol AKE_Device:Test_Point
Connections:
- net GND: now also C102.1, D45.1, SW3.3, SW3.4
- new net: D45.2, R98.2
- new net +3.3V_MCU: R103.2
- new net User_Button: C102.2, R103.1, SW3.1, SW3.2
- new net User_Led: R98.1, TP33.1

Commit message: 12.01.2025
Changed lines of the file:
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@@
 			(effects
 				(font
-					(size 1.27 1.27)
+					(face "Arial")
+					(size 0.635 0.635)
 				)
 				(hide yes)
@@
 			(effects
 				(font
-					(size 1.27 1.27)
+					(face "Arial")
+					(size 0.635 0.635)
 				)
 				(justify left)
@@
 			(effects
 				(font
-					(size 1.27 1.27)
+					(face "Arial")
+					(size 0.635 0.635)
 				)
 				(hide yes)
@@
 			(effects
 				(font
-					(size 1.27 1.27)
+					(face "Arial")
+					(size 0.635 0.635)
 				)
 				(hide yes)
@@
 			(effects
 				(font
-					(size 1.27 1.27)
+					(face "Arial")
+					(size 0.635 0.635)
 				)
 				(justify right)
@@
 			(effects
 				(font
-					(size 1.27 1.27)
+					(face "Arial")
+					(size 0.635 0.635)
 				)
 			)
@@
 			(effects
 				(font
-					(size 1.27 1.27)
+					(face "Arial")
+					(size 0.635 0.635)
 				)
 				(justify left)
@@
 			(effects
 				(font
-					(size 1.27 1.27)
+					(face "Arial")
+					(size 0.635 0.635)
 				)
 				(hide yes)
@@
 			(effects
 				(font
-					(size 1.27 1.27)
+					(face "Arial")
+					(size 0.635 0.635)
 				)
 				(justify right)
@@
 			(effects
 				(font
-					(size 1.27 1.27)
-				)
-			)
+					(face "Arial")
+					(size 0.635 0.635)
+				)
+			)
